File: hardware/extensioncard/extensioncard.kicad_pcb (KiCad board)
At the start: 2 copper layers, 203.2 x 63.5 mm, 3 parts, among them J1 Male Card Edge, J2 Header, J3 Female Card Edge

Commit message: extensioncard hopefully done
Parts:
- removed the J2 at (50.8, 100.4)
- added J3: Header, Connector_PinHeader_2.54mm:PinHeader_2x15_P2.54mm_Vertical, F.Cu at (48.3, 119.4)
- moved J1 19.0 mm to (241.3, 101.6)
- moved J2 19.0 mm to (63.5, 101.6)
- renumbered J3 to J2
Routing:
- net /PIN15: track 201.4 -> 192.1 mm
- net /PIN1: track 189.8 -> 195.0 mm
- net /PIND: track 192.0 -> 196.4 mm
- net /PINE: track 191.4 -> 195.7 mm
- net /PIN3: track 188.4 -> 192.6 mm
- net /PIN2: track 189.0 -> 193.2 mm
- net /PINB: track 193.2 -> 197.3 mm
- net /PINF: track 190.8 -> 194.9 mm
- net /PINP: track 192.8 -> 196.8 mm
- net /PIN7: track 186.5 -> 190.2 mm
- net /PINC: track 192.6 -> 195.9 mm
- net /PINN: track 192.3 -> 195.6 mm
- net /PINR: track 193.5 -> 196.7 mm
- net /PINM: track 191.7 -> 195.0 mm
- net /PINL: track 191.5 -> 194.6 mm
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- removed copper zone on B.Cu, net (none)
Other:
- outline, holes or cut-outs redrawn
- board text added: "10"
- board text added: "11"
- board text added: "12"
- board text added: "13"
- board text added: "14"
- board text added: "2"
- board text added: "3"
- board text added: "4"
- board text added: "5"
- board text added: "6"
- board text added: "7"
- board text added: "8"
- board text added: "9"
- board text added: "B"
- board text added: "C"
- board text added: "COMPONENT SIDE"
- board text added: "D"
- board text added: "E"
- board text added: "F"
- board text added: "H"
- board text added: "J"
- board text added: "JLCJLCJLCJLC"
- board text added: "K"
- board text added: "L"
- board text added: "M"
- board text added: "N"
- board text added: "P"
- board text added: "R"
- board text added: "SOLDER SIDE"
- board text added: "WANG 2200 EXTENSION CARD"
- board text added: "©2021 DENZ@HACK42"

Commit message: upcycled to newer version KiCad
Other:
- net class Default removed
