File: hardware/powerprobe/powerprobe.kicad_pcb (KiCad board)
At the start: 2 copper layers, 47 x 88.9 mm, 16 parts, among them J1 CONN1, J2 CONN2

Commit message: upcycled to newer version KiCad
Other:
- net class Default removed
