File: hardware/heatsink/heatsink.kicad_sch (KiCad schematic)
At the start: 2 parts, among them J1 Heatsink, J2 Heatsink

Commit message: small update in schematic
Other:
- sheet -12VR ports: added -12VR, 0V, B1-12R, B2-12R; removed none
